File: hw/sch_pcb/GLCD01.kicad_pcb (KiCad board)
At the start: 2 copper layers, 40.1 x 40.1 mm, 8 parts, among them J1 Umin ... Umax, M1 HOLE M3, M2 HOLE M3, M3 HOLE, M4 HOLE

Commit message: v1 with mic1557
Parts:
- removed C1: 10uF, Capacitor_SMD:C_0805_2012Metric
- removed D1: BZV55C-5,6V, Diode_SMD:D_SMA
- added C3: 100nF/63V, Capacitor_SMD:C_0603_1608Metric, F.Cu at (124.3, 102.4)
- added C4: 100nF/63V, Capacitor_SMD:C_0603_1608Metric, F.Cu at (132.1, 97.7)
- added J2: 046824610000846+, FPC:046824610000846, F.Cu at (127.1, 107.2)
- added Q1: BSS138, Package_TO_SOT_SMD:SOT-23, F.Cu at (135.9, 95.5)
- added R1: 750k, Resistor_SMD:R_0603_1608Metric, F.Cu at (133.1, 104.6)
- added R2: 1M, Resistor_SMD:R_0603_1608Metric, F.Cu at (132.1, 95.4)
- added R3: 1k, Resistor_SMD:R_0603_1608Metric, F.Cu at (136.0, 91.5)
- added R4: 1M, Resistor_SMD:R_0603_1608Metric, F.Cu at (137.1, 100.5)
- added U1: MIC1557YM5-TR, Package_TO_SOT_SMD:SOT-23-5, F.Cu at (133.0, 100.6)
- C2: value 100nF -> GRM21BR71H105KA12L; footprint Capacitor_SMD:C_0805_2012Metric -> Capacitor_SMD:C_0603_1608Metric; moved to F.Cu
- J1: value Umin ... Umax -> JUMP_7X2; footprint Mlab_Pin_Headers:Straight_2x03 -> Mlab_Pin_Headers:Straight_2x07
- moved C2 23.8 mm to (136.7, 104.6), turned to 0 degrees
- moved J1 21.8 mm to (126.7, 81.3), turned to 90 degrees
Connections:
- C2 pad 1: +5V -> Net-(U1-T/T)
- J1 pad 1: GND -> +3.3V
- J1 pad 2: GND -> +3.3V
- J1 pad 3: +5V -> Net-(J1-4-Pad3)
- J1 pad 4: +5V -> Net-(J1-4-Pad3)
- J1 pad 5: GND -> Net-(J1-6-Pad5)
- J1 pad 6: GND -> Net-(J1-6-Pad5)
Routing:
- net +3.3V: track 0.00 -> 0.87 mm
- net Net-(J1-6-Pad5): track 0.00 -> 0.59 mm
- net GND: track 0.00 -> 0.59 mm
- net Net-(J1-4-Pad3): track 0.00 -> 0.57 mm
- net Net-(J1-8-Pad7): track 0.00 -> 0.56 mm
- net Net-(J1-10-Pad9): track 0.00 -> 0.55 mm
